File: PCB/starlink-apo-pcb.kicad_pcb (KiCad board)
At the start: 2 copper layers, 55.1 x 15.5 mm, 29 parts, among them J1 Barrel_Jack, J2 Barrel_Jack, Q1 CSD16327Q3, Q2 CSD16327Q3, U1 TPS43061RTE

Commit message: v0.0.1 off to JLCPCB
Parts:
- removed C3: 22uF 50V, Capacitor_SMD:C_1812_4532Metric
- added D1: LED_Small, LED_SMD:LED_0402_1005Metric, F.Cu at (155.3, 68.1)
- added R9: 11kR, Resistor_SMD:R_0603_1608Metric, F.Cu at (143.3, 67.9)
- C4: value 22uF 50V -> 10uF 50V; footprint Capacitor_SMD:C_1812_4532Metric -> Capacitor_SMD:C_1210_3225Metric
- C5: value 22uF 50V -> 33uF 50V; footprint Capacitor_SMD:C_1812_4532Metric -> Capacitor_SMD:C_Elec_6.3x7.7
- moved C4 7.61 mm to (141.3, 71.2)
- moved C5 7.34 mm to (141.4, 77.5), turned to -90 degrees
- moved C1 5.85 mm to (126.2, 74.0)
- moved R1 1.15 mm to (123.9, 74.6)
- moved R2 0.46 mm to (128.5, 74.6)
Connections:
- C1 pad 1: Net-(C1-Pad1) -> ISNS-
- L1 pad 1: Net-(U1-ISNS–) -> Net-(L1-Pad1)
- R2 pad 1: Net-(C1-Pad1) -> ISNS-
- R2 pad 2: Net-(U1-ISNS–) -> Net-(L1-Pad1)
- R3 pad 1: Net-(U1-ISNS–) -> Net-(L1-Pad1)
- R5 pad 1: Net-(U1-ISNS–) -> Net-(L1-Pad1)
- U1 pad 5: Net-(U1-ISNS–) -> ISNS-
Routing:
- net Net-(D1-K): track 0.00 -> 12.2 mm
- net Net-(C1-Pad1): track 10.8 -> 0.00 mm, vias 2 -> 0
- net ISNS-: track 0.00 -> 6.66 mm, vias 0 -> 2
- net Net-(U1-ISNS–): track 6.42 -> 0.00 mm, vias 22 -> 0
- net ISNS+: track 8.82 -> 4.03 mm, vias 2 -> 0
- net Net-(U1-VIN): track 6.31 -> 7.81 mm, vias 19 -> 20
- net Net-(D1-A): track 96.5 -> 95.5 mm
- net Net-(L1-Pad1): vias 0 -> 14
- net GND: vias 129 -> 126
- added copper zone on B.Cu, net Net-(L1-Pad1)
- added copper zone on F.Cu, net Net-(L1-Pad1)
- removed copper zone on B.Cu, net Net-(U1-ISNS–)
- removed copper zone on F.Cu, net Net-(U1-ISNS–)
Other:
- board text added: "JLCJLCJLCJLC"
