File: PCB/starlink-apo-pcb.kicad_sch (KiCad schematic)
At the start: 27 parts, among them J1 Barrel_Jack, J2 Barrel_Jack, Q1 CSD16327Q3, Q2 CSD16327Q3, U1 TPS43061RTE

Commit message: v0.0.1 off to JLCPCB
Parts:
- removed C3: 22uF 50V, Capacitor_SMD:C_1812_4532Metric, symbol Device:C_Small
- added D1: LED_Small, LED_SMD:LED_0402_1005Metric, symbol Device:LED_Small
- added R9: 11kR, Resistor_SMD:R_0603_1608Metric, symbol Device:R_Small
- C1: LCSC (none) -> C14858
- C10: LCSC (none) -> C96446
- C11: LCSC (none) -> C1608
- C12: LCSC (none) -> C1604
- C13: LCSC (none) -> C53987
- C2, C9: LCSC (none) -> C14663
- C4: value 22uF 50V -> 10uF 50V; footprint Capacitor_SMD:C_1812_4532Metric -> Capacitor_SMD:C_1210_3225Metric; LCSC (none) -> C138687; lcsc C22388553 -> C138687
- C5: value 22uF 50V -> 33uF 50V; footprint Capacitor_SMD:C_1812_4532Metric -> Capacitor_SMD:C_Elec_6.3x7.7; symbol Device:C_Small -> Device:C_Polarized_Small; LCSC (none) -> C402500; lcsc C22388553 -> C402500
- C6, C7, C8: LCSC (none) -> C138687
- J1, J2: LCSC (none) -> C3096082
- L1: LCSC (none) -> C19191671
- Q1, Q2: LCSC (none) -> C840100
- R1, R2: LCSC (none) -> C22775
- R3, R5: LCSC (none) -> C1021507
- R4: LCSC (none) -> C5126104
- R6: LCSC (none) -> C25950
- R7: LCSC (none) -> C228022
- R8: LCSC (none) -> C2933128
- U1: LCSC (none) -> C527683; lcsc C3188675 -> C527683
Connections:
- net GND: now also R9.2
- net at C4.1, C5.1, J2.1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: now also D1.2 (A)
- net ISNS-: now reaches C1.1, R2.1
- net ISNS-: now also U1.5 (ISNS–)
- net at L1.1, R2.2, R3.1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: no longer U1.5 (ISNS–)
- new net: D1.1 (K), R9.1
Other:
- note added: "16V 6A resettable fuse: C910847 30V 2.6A resettable fuse: C41367375"
- moved on the sheet: C4, J2
